File: meshcore-solar.kicad_pcb (KiCad board)
At the start: 2 copper layers, 58.1 x 89 mm, 44 parts, among them P1 PH2.0-2P-LT, SW1 Tactile Button, 160gf, U1 RAK4630-8-SM-I, U2 SGM41513YTQF24G/TR, U3 XC6206P332MR

Commit message: Board rev B: fixes, low-voltage cutoff, SMT holder, USB override
Schematic fixes after datasheet review:
- Battery sense moved to P0.05/AIN3 with 1M/1.5M divider (stock MeshCore RAK4631)
- I2C pull-ups moved to VDD_NRF (nRF I/O rail)

New features:
- Hardware low-voltage cutoff (MCP65R41 + TPS22917): SYS_SW off below ~3.30 V,
  back on above ~3.73 V; JP1 bench bypass
- USB VBUS forces the cutoff on (D3/R15/R16) so the RAK can always be flashed
  over USB, even with no cell
- SMT 18650 holder MYOUNG BH-18650-B1BA002 (C2988620); footprint and 3D model
  generated with kicad-library-tools, sources in library-src/

Layout:
- Board 58.1 x 91.0 mm (top edge +2.3 mm for holder/mounting-hole clearance)
- 45-degree chamfers on all right-angle track bends; teardrops on vias/THT pads
- Project-local 3D models for U4/U5, D3, L1 and the holder

Tooling: scripts/export.sh for ERC/DRC and JLCPCB outputs.

Co-Authored-By: Claude Opus 5.5 <noreply@anthropic.com>
Parts:
- added C16: 100nF, PCM_JLCPCB:C_0805, F.Cu at (136.1, 91.7)
- added C17: 100nF, PCM_JLCPCB:C_0805, F.Cu at (144.1, 88.0)
- added D3: 1N4148W, Diode_SMD:D_SOD-123, F.Cu at (130.2, 94.0)
- added JP1: Bypass, Jumper:SolderJumper-2_P1.3mm_Open_RoundedPad1.0x1.5mm, F.Cu at (130.4, 90.2)
- added R12: 390kΩ, PCM_JLCPCB:R_0805, F.Cu at (144.1, 84.5)
- added R13: 200kΩ, PCM_JLCPCB:R_0805, F.Cu at (144.1, 91.5)
- added R14: 3MΩ, PCM_JLCPCB:R_0805, F.Cu at (141.6, 88.2)
- added R15: 100kΩ, PCM_JLCPCB:R_0805, F.Cu at (140.0, 92.4)
- added R16: 10kΩ, PCM_JLCPCB:R_0805, F.Cu at (130.2, 98.9)
- added U4: MCP65R41, Package_TO_SOT_SMD:SOT-23-6, F.Cu at (137.2, 88.2)
- added U5: TPS22917, Package_TO_SOT_SMD:SOT-23-6, F.Cu at (130.4, 87.2)
- BT1: value BH-18650-A1AJ005 -> BH-18650-B1BA002; footprint lcsc_shared_footprints:C5290176_BAT-TH_BH-18650-A1AJ005 -> meshcore-solar:BatteryHolder_MYOUNG_BH-18650-B1BA002_1x18650
- R11: value 1MΩ -> 1.5MΩ
- moved H1 2.30 mm to (97.4, 34.7)
- moved H2 2.30 mm to (148.5, 34.7)
- moved BT1 1.15 mm to (105.4, 76.8)
- turned C15 to 90 degrees
Connections:
- BT1 pad 1: GND -> +BATT
- BT1 pad 2: +BATT -> GND
- C10 pad 1: /SYS -> /SYS_SW
- C11 pad 1: /SYS -> /SYS_SW
- R4 pad 1: +3V3 -> /VDD_NRF
- R5 pad 1: +3V3 -> /VDD_NRF
- U1 pad 39: /VBAT_SENSE -> unconnected-(U1-P0.31/AIN7-Pad39)
- U1 pad 40: unconnected-(U1-P0.05/AIN3-Pad40) -> /VBAT_SENSE
- U1 pad 44: /SYS -> /SYS_SW
- U3 pad 3: /SYS -> /SYS_SW
Routing:
- net /SYS_SW: track 0.00 -> 56.7 mm, vias 0 -> 2
- net +BATT: track 63.6 -> 116.2 mm, vias 3 -> 6
- net /SYS: track 45.0 -> 21.1 mm, vias 2 -> 0
- net Net-(D3-K): track 0.00 -> 22.3 mm, vias 0 -> 3
- net /VDD_NRF: track 86.7 -> 104.0 mm, vias 3 -> 5
- net +3V3: track 46.1 -> 29.3 mm, vias 4 -> 2
- net GND: track 39.5 -> 53.8 mm, vias 80 -> 77
- net Net-(U4-+): track 0.00 -> 12.7 mm
- net /CUTOFF_EN: track 0.00 -> 5.61 mm
- net VBUS: track 86.0 -> 90.9 mm
- net Net-(D3-A): track 0.00 -> 2.34 mm
- net /VBUS_IN: track 44.1 -> 42.1 mm
- net /REGN: track 38.0 -> 36.4 mm
- net Net-(U4--): track 0.00 -> 0.95 mm
- net /NTC: track 25.6 -> 24.9 mm
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Other:
- board size 58.1 x 89 mm -> 58.1 x 91.3 mm
