File: meshcore-solar.kicad_sch (KiCad schematic)
At the start: 40 parts, among them P1 PH2.0-2P-LT, SW1 Tactile Button, 160gf, U1 RAK4630-8-SM-I, U2 SGM41513YTQF24G/TR, U3 XC6206P332MR

Commit message: Board rev B: fixes, low-voltage cutoff, SMT holder, USB override
Schematic fixes after datasheet review:
- Battery sense moved to P0.05/AIN3 with 1M/1.5M divider (stock MeshCore RAK4631)
- I2C pull-ups moved to VDD_NRF (nRF I/O rail)

New features:
- Hardware low-voltage cutoff (MCP65R41 + TPS22917): SYS_SW off below ~3.30 V,
  back on above ~3.73 V; JP1 bench bypass
- USB VBUS forces the cutoff on (D3/R15/R16) so the RAK can always be flashed
  over USB, even with no cell
- SMT 18650 holder MYOUNG BH-18650-B1BA002 (C2988620); footprint and 3D model
  generated with kicad-library-tools, sources in library-src/

Layout:
- Board 58.1 x 91.0 mm (top edge +2.3 mm for holder/mounting-hole clearance)
- 45-degree chamfers on all right-angle track bends; teardrops on vias/THT pads
- Project-local 3D models for U4/U5, D3, L1 and the holder

Tooling: scripts/export.sh for ERC/DRC and JLCPCB outputs.

Co-Authored-By: Claude Opus 5.5 <noreply@anthropic.com>
Parts:
- removed BT1: BH-18650-A1AJ005, lcsc_shared_footprints:C5290176_BAT-TH_BH-18650-A1AJ005, symbol LCSC:BH-18650-A1AJ005
- added BT1: BH-18650-B1BA002, meshcore-solar:BatteryHolder_MYOUNG_BH-18650-B1BA002_1x18650, symbol Device:Battery_Cell
- added C16, C17: 100nF, PCM_JLCPCB:C_0805, symbol PCM_JLCPCB-Capacitors:0805,100nF
- added D3: 1N4148W, Diode_SMD:D_SOD-123, symbol Device:D
- added JP1: Bypass, Jumper:SolderJumper-2_P1.3mm_Open_RoundedPad1.0x1.5mm, symbol Jumper:SolderJumper_2_Open
- added R12: 390kΩ, PCM_JLCPCB:R_0805, symbol PCM_JLCPCB-Resistors:0805,10kΩ
- added R13: 200kΩ, PCM_JLCPCB:R_0805, symbol PCM_JLCPCB-Resistors:0805,10kΩ
- added R14: 3MΩ, PCM_JLCPCB:R_0805, symbol PCM_JLCPCB-Resistors:0805,10kΩ
- added R15: 100kΩ, PCM_JLCPCB:R_0805, symbol PCM_JLCPCB-Resistors:0805,10kΩ
- added R16: 10kΩ, PCM_JLCPCB:R_0805, symbol PCM_JLCPCB-Resistors:0805,10kΩ
- added U4: MCP65R41, Package_TO_SOT_SMD:SOT-23-6, symbol meshcore-solar:MCP65R41
- added U5: TPS22917, Package_TO_SOT_SMD:SOT-23-6, symbol meshcore-solar:TPS22917DBV
- R11: value 1MΩ -> 1.5MΩ; Class Basic Component -> Extended Component; LCSC C17514 -> C26110; Part 0805W8F1004T5E -> 0805W8F1504T5E; Resistance 1MΩ -> 1.5MΩ; Stock 859014 -> 26100
Connections:
- net +3V3: no longer R4.1, R5.1
- net +BATT: now also BT1.1 (+), C16.1, R12.1, U4.6 (V+)
- net GND: now also BT1.2 (-), C16.2, C17.2, R13.2, U4.2 (V-), U5.2 (GND)
- net SYS: now also JP1.1 (A), U5.1 (VIN); no longer C10.1, C11.1, U1.44 (VBAT_NRF), U3.3 (VIN)
- net VBAT_SENSE: now also U1.40 (P0.05/AIN3); no longer U1.39 (P0.31/AIN7)
- net VBUS: now also R16.1
- net VDD_NRF: now also R4.1, R5.1
- new net: D3.1 (K), R15.2, U5.3 (ON)
- new net: C17.1, R12.2, R13.1, R14.1, U4.3 (+)
- new net: U4.4 (-), U4.5 (Vref)
- new net: D3.2 (A), R16.2
- new net CUTOFF_EN: R14.2, R15.1, U4.1
- new net SYS_SW: C10.1, C11.1, JP1.2 (B), U1.44 (VBAT_NRF), U3.3 (VIN), U5.5 (QOD), U5.6 (VOUT)
- no-connect marks 32 -> 33
Other:
- note added: "BAT falling < 3.30 V: SYS_SW off BAT rising > 3.73 V: SYS_SW on"
- note added: "CT open: fastest turn-on (~65 us), OK for the ~6 uF on SYS_SW"
- note added: "LOW-VOLTAGE CUTOFF"
- note added: "USB present: D3 forces SYS_SW on. JP1: bypass (no USB, no cell)"
